Commit message: Update robot.xacro

File: urdf/robot.xacro (robot description, xacro)
@@ -3,27 +3,9 @@
   <xacro:include filename="$(find task_6)/urdf/robot.gazebo" />
   <!-- materials -->
-  <material name="black">
-    <color rgba="0.0 0.0 0.0 1.0"/>
-  </material>
   <material name="blue">
     <color rgba="0.203125 0.23828125 0.28515625 1.0"/>
   </material>
-  <material name="green">
-    <color rgba="0.0 0.8 0.0 1.0"/>
-  </material>
-  <material name="grey">
-    <color rgba="0.2 0.2 0.2 1.0"/>
-  </material>
   <material name="orange">
     <color rgba="1.0 0.423529411765 0.0392156862745 1.0"/>
-  </material>
-  <material name="brown">
-    <color rgba="0.870588235294 0.811764705882 0.764705882353 1.0"/>
-  </material>
-  <material name="red">
-    <color rgba="0.80078125 0.12890625 0.1328125 1.0"/>
-  </material>
-  <material name="white">
-    <color rgba="1.0 1.0 1.0 1.0"/>
   </material>
   <!-- macros -->
